Commit message: Add MoveIt launch for the real arm and handover docs
moveit_real.launch.py starts xarm's Lite 6 MoveIt with the arm pose from
arm_platform.yaml, composing platform and arm pose and quoting the attach
arguments the way xarm's launch expects.

The platform pose is now xyz/rpy instead of a height, so the same keys
place the platform on the Amiga later. README covers running the arm on
the Orin, adjusting the mount and troubleshooting.

File: src/amiga_description/urdf/arm_platform_standalone.urdf.xacro (robot description, xacro)
@@ -1,5 +1,5 @@
 <?xml version="1.0"?>
 <robot name="arm_platform" xmlns:xacro="http://ros.org/wiki/xacro">
-  <!-- The arm platform on its own, fixed to the world at rail height. -->
+  <!-- The arm platform on its own, fixed to the world (floor) at platform xyz/rpy from the config. -->
   <xacro:arg name="config" default="$(find amiga_description)/config/arm_platform.yaml"/>
   <xacro:arg name="ros2_control_plugin" default="uf_robot_hardware/UFRobotSystemHardware"/>
@@ -7,6 +7,7 @@
   <xacro:include filename="$(find amiga_description)/urdf/arm_platform.xacro"/>
   <link name="world"/>
+  <xacro:property name="platform" value="${xacro.load_yaml('$(arg config)')['platform']}"/>
   <xacro:arm_platform parent="world"
-    xyz="0 0 ${xacro.load_yaml('$(arg config)')['platform']['height']}" rpy="0 0 0"
+    xyz="${' '.join(map(str, platform['xyz']))}" rpy="${' '.join(map(str, platform['rpy']))}"
     config="$(arg config)"
     ros2_control_plugin="$(arg ros2_control_plugin)"
