Commit message: Drive the Amiga in Gazebo with cmd_vel
gazebo.launch.py spawns the Amiga free on the ground with
amiga_description's Gazebo drive (v0.5.0) and bridges /cmd_vel,
/wheel/odometry, the wheel joint states and optionally the odom TF.
amiga_arm.urdf.xacro gets fixed and gazebo arguments. Keyboard teleop
in the image; simulation docs written for students.

File: src/amiga_arm_description/urdf/amiga_arm.urdf.xacro (robot description, xacro)
@@ -2,16 +2,25 @@
 <robot name="amiga_arm" xmlns:xacro="http://ros.org/wiki/xacro">
   <!-- The Amiga with the arm platform on its base_link (platform xyz/rpy from the config).
-       The Amiga stands fixed on "world" (the floor): MoveIt and Gazebo use world as the root. -->
+       fixed:=true   the Amiga stands fixed on "world" (the floor), the root for RViz and MoveIt
+       gazebo:=true  adds the Gazebo drive (use with fixed:=false, so the Amiga can drive) -->
   <xacro:arg name="config" default="$(find amiga_arm_description)/config/arm_platform.yaml"/>
   <xacro:arg name="ros2_control_plugin" default="uf_robot_hardware/UFRobotSystemHardware"/>
   <xacro:arg name="robot_ip" default="10.95.76.155"/>
+  <xacro:arg name="fixed" default="true"/>
+  <xacro:arg name="gazebo" default="false"/>
   <xacro:include filename="$(find amiga_description)/urdf/amiga.xacro"/>
   <xacro:include filename="$(find amiga_arm_description)/urdf/arm_platform.xacro"/>
-  <link name="world"/>
-  <joint name="world_to_amiga_joint" type="fixed">
-    <parent link="world"/>
-    <child link="base_footprint"/>
-  </joint>
+  <xacro:if value="$(arg fixed)">
+    <link name="world"/>
+    <joint name="world_to_amiga_joint" type="fixed">
+      <parent link="world"/>
+      <child link="base_footprint"/>
+    </joint>
+  </xacro:if>
   <xacro:amiga prefix=""/>
+  <xacro:if value="$(arg gazebo)">
+    <xacro:include filename="$(find amiga_description)/urdf/amiga.gazebo.xacro"/>
+    <xacro:amiga_gazebo prefix=""/>
+  </xacro:if>
   <xacro:property name="platform" value="${xacro.load_yaml('$(arg config)')['platform']}"/>
   <xacro:arm_platform parent="base_link"

Commit message: Pick a pixelfield carrot in simulation
Sideways arm mount (arm_sideways in arm_platform.yaml, launch arg
sideways), Gripper Lite with a gripper_controller (gripper:=true),
spawn pose args x/y/yaw, and the arm platform on collide bit 0x1 so it
passes through pixelfield Plants.

The gripper uses xarm's links with an own ros2_control block: xarm's
add_gripper mimics finger 2 through a plugin that does not load in gz
sim, while gz_ros2_control mimics it from the URDF.

The image gets pixelfield (AgriSim daed17a) and its pull-out system.
scripts/pick_carrot.py takes a carrot from the Field's manifest, moves
the gripper down onto its leaf bunch, closes it and lifts by the root
length, then reports what the Plant did. With the modelled 5 N grip
the carrot passes its Pull-out Force but slips before it comes free.

File: src/amiga_arm_description/urdf/amiga_arm.urdf.xacro (robot description, xacro)
@@ -3,5 +3,7 @@
   <!-- The Amiga with the arm platform on its base_link (platform xyz/rpy from the config).
        fixed:=true   the Amiga stands fixed on "world" (the floor), the root for RViz and MoveIt
-       gazebo:=true  adds the Gazebo drive (use with fixed:=false, so the Amiga can drive) -->
+       gazebo:=true  adds the Gazebo drive (use with fixed:=false, so the Amiga can drive)
+       sideways:=true  arm pose from `arm_sideways` in the config instead of `arm`
+       gripper:=true  adds the Gripper Lite (simulation: its controller is in sim_controllers.yaml) -->
   <xacro:arg name="config" default="$(find amiga_arm_description)/config/arm_platform.yaml"/>
   <xacro:arg name="ros2_control_plugin" default="uf_robot_hardware/UFRobotSystemHardware"/>
@@ -9,4 +11,6 @@
   <xacro:arg name="fixed" default="true"/>
   <xacro:arg name="gazebo" default="false"/>
+  <xacro:arg name="sideways" default="false"/>
+  <xacro:arg name="gripper" default="false"/>
   <xacro:include filename="$(find amiga_description)/urdf/amiga.xacro"/>
   <xacro:include filename="$(find amiga_arm_description)/urdf/arm_platform.xacro"/>
@@ -26,5 +30,6 @@
   <xacro:arm_platform parent="base_link"
     xyz="${' '.join(map(str, platform['xyz']))}" rpy="${' '.join(map(str, platform['rpy']))}"
-    config="$(arg config)"
+    config="$(arg config)" arm_key="${'arm_sideways' if '$(arg sideways)'.lower() in ('true', '1') else 'arm'}"
+    gripper="$(arg gripper)"
     ros2_control_plugin="$(arg ros2_control_plugin)"
     robot_ip="$(arg robot_ip)"/>

File: src/amiga_arm_description/urdf/arm_platform.xacro (robot description, xacro)
@@ -4,5 +4,5 @@
        platform_link origin: top front edge of the Amiga cross tube the top plank rests on.
        Geometry and arm pose come from config/arm_platform.yaml. -->
-  <xacro:macro name="arm_platform" params="parent xyz rpy config ros2_control_plugin robot_ip">
+  <xacro:macro name="arm_platform" params="parent xyz rpy config arm_key gripper ros2_control_plugin robot_ip">
     <xacro:property name="cfg" value="${xacro.load_yaml(config)}"/>
     <xacro:property name="plank" value="${cfg['platform']['plank']}"/>
@@ -10,5 +10,5 @@
     <xacro:property name="W" value="${plank['width']}"/>
     <xacro:property name="T" value="${plank['thickness']}"/>
-    <xacro:property name="arm" value="${cfg['arm']}"/>
+    <xacro:property name="arm" value="${cfg[arm_key]}"/>
     <material name="plank_wood">
       <color rgba="0.76 0.60 0.42 1.0"/>
@@ -36,4 +36,9 @@
       </inertial>
     </link>
+    <!-- Collide bit 0 only: the planks touch the soil and the Amiga, but no pixelfield Plant
+         (robot interface 2), so they neither pick nor crush Plants under the platform. -->
+    <gazebo reference="platform_link">
+      <collision><surface><contact><collide_bitmask>0x01</collide_bitmask></contact></surface></collision>
+    </gazebo>
     <joint name="platform_joint" type="fixed">
       <parent link="${parent}"/>
@@ -47,5 +52,28 @@
       attach_rpy="${' '.join(map(str, arm['rpy']))}"
       ros2_control_plugin="${ros2_control_plugin}" load_gazebo_plugin="true"
+      ros2_control_params="${'$(find amiga_arm_description)/config/sim_controllers.yaml' if gripper else ''}"
       robot_ip="${robot_ip}"/>
+    <!-- Gripper Lite: xarm's links and joints, but not its add_gripper. That one makes finger 2
+         follow finger 1 through a Gazebo Classic style plugin that does not load in gz sim, so
+         here gz_ros2_control mimics finger_joint2 (its URDF <mimic>) instead. -->
+    <xacro:if value="${gripper}">
+      <xacro:include filename="$(find xarm_description)/urdf/common/common.link.xacro"/>
+      <xacro:include filename="$(find xarm_description)/urdf/gripper/uflite_gripper.urdf.xacro"/>
+      <xacro:uflite_gripper_urdf attach_to="link_eef"/>
+      <xacro:if value="${ros2_control_plugin == 'gz_ros2_control/GazeboSimSystem'}">
+        <ros2_control name="GripperLiteSystem" type="system">
+          <hardware><plugin>${ros2_control_plugin}</plugin></hardware>
+          <joint name="finger_joint1">
+            <command_interface name="position"/>
+            <command_interface name="velocity"/>
+            <state_interface name="position"/>
+            <state_interface name="velocity"/>
+          </joint>
+          <joint name="finger_joint2">
+            <state_interface name="position"/>
+          </joint>
+        </ros2_control>
+      </xacro:if>
+    </xacro:if>
   </xacro:macro>
 </robot>

Commit message: Simulate an xArm 6 option that pulls a carrot out
- robot:=xarm6: xArm 6 with the xArm Gripper as two effort-controlled
  parallel jaws (30 N each, xarm meshes); the Lite 6 stays the default.
- sideways:=true: arm on the vertical plank, pointing forward, reaching
  the soil between the axles; the real pose is unchanged.
- pick_carrot.py: Amiga straddles a bed of amiga_10x10, sim-time
  gripper waits, gripper effort per robot.
- Arm links pass through pixelfield Plants (collide bit 0x1), so a
  dense bed no longer stalls the simulation.
- fields/crops/carrot.yaml: carrots 10 cm apart in the row; at 4 cm
  the jaws grab the neighbours' leaves instead of the target.

File: src/amiga_arm_description/urdf/amiga_arm.urdf.xacro (robot description, xacro)
@@ -4,6 +4,7 @@
        fixed:=true   the Amiga stands fixed on "world" (the floor), the root for RViz and MoveIt
        gazebo:=true  adds the Gazebo drive (use with fixed:=false, so the Amiga can drive)
-       sideways:=true  arm pose from `arm_sideways` in the config instead of `arm`
-       gripper:=true  adds the Gripper Lite (simulation: its controller is in sim_controllers.yaml) -->
+       robot:=xarm6  an xArm 6 instead of the Lite 6 (simulation option), pose from `xarm6` in the config
+       sideways:=true  arm (and platform) pose from `<pose>_sideways` in the config: arm points forward
+       gripper:=true  adds the arm's gripper (simulation: its controller is in sim_controllers.yaml) -->
   <xacro:arg name="config" default="$(find amiga_arm_description)/config/arm_platform.yaml"/>
   <xacro:arg name="ros2_control_plugin" default="uf_robot_hardware/UFRobotSystemHardware"/>
@@ -11,4 +12,5 @@
   <xacro:arg name="fixed" default="true"/>
   <xacro:arg name="gazebo" default="false"/>
+  <xacro:arg name="robot" default="lite6"/>
   <xacro:arg name="sideways" default="false"/>
   <xacro:arg name="gripper" default="false"/>
@@ -27,8 +29,12 @@
     <xacro:amiga_gazebo prefix=""/>
   </xacro:if>
-  <xacro:property name="platform" value="${xacro.load_yaml('$(arg config)')['platform']}"/>
+  <xacro:property name="cfg" value="${xacro.load_yaml('$(arg config)')}"/>
+  <xacro:property name="arm_key"
+    value="${('arm' if '$(arg robot)' == 'lite6' else '$(arg robot)') + ('_sideways' if '$(arg sideways)'.lower() in ('true', '1') else '')}"/>
+  <!-- An arm pose can bring its own platform pose (the sideways mounts) -->
+  <xacro:property name="platform" value="${cfg[arm_key].get('platform', cfg['platform'])}"/>
   <xacro:arm_platform parent="base_link"
     xyz="${' '.join(map(str, platform['xyz']))}" rpy="${' '.join(map(str, platform['rpy']))}"
-    config="$(arg config)" arm_key="${'arm_sideways' if '$(arg sideways)'.lower() in ('true', '1') else 'arm'}"
+    config="$(arg config)" robot="$(arg robot)" arm_key="${arm_key}"
     gripper="$(arg gripper)"
     ros2_control_plugin="$(arg ros2_control_plugin)"

File: src/amiga_arm_description/urdf/arm_platform.xacro (robot description, xacro)
@@ -1,8 +1,8 @@
 <?xml version="1.0"?>
 <robot xmlns:xacro="http://ros.org/wiki/xacro">
-  <!-- Two planks screwed together at 90 degrees, with a Lite 6 on the vertical one.
+  <!-- Two planks screwed together at 90 degrees, with a UFactory arm (robot: lite6 or xarm6).
        platform_link origin: top front edge of the Amiga cross tube the top plank rests on.
        Geometry and arm pose come from config/arm_platform.yaml. -->
-  <xacro:macro name="arm_platform" params="parent xyz rpy config arm_key gripper ros2_control_plugin robot_ip">
+  <xacro:macro name="arm_platform" params="parent xyz rpy config robot arm_key gripper ros2_control_plugin robot_ip">
     <xacro:property name="cfg" value="${xacro.load_yaml(config)}"/>
     <xacro:property name="plank" value="${cfg['platform']['plank']}"/>
@@ -41,4 +41,17 @@
       <collision><surface><contact><collide_bitmask>0x01</collide_bitmask></contact></surface></collision>
     </gazebo>
+    <!-- The arm links as well: leaves push only on the gripper. Arm links in a dense bed pick
+         and push dozens of Plants, which slows the simulation down to a few percent of real time. -->
+    <xacro:macro name="soil_only" params="link">
+      <gazebo reference="${link}">
+        <collision><surface><contact><collide_bitmask>0x01</collide_bitmask></contact></surface></collision>
+      </gazebo>
+    </xacro:macro>
+    <xacro:soil_only link="link1"/>
+    <xacro:soil_only link="link2"/>
+    <xacro:soil_only link="link3"/>
+    <xacro:soil_only link="link4"/>
+    <xacro:soil_only link="link5"/>
+    <xacro:soil_only link="link6"/>
     <joint name="platform_joint" type="fixed">
       <parent link="${parent}"/>
@@ -47,5 +60,5 @@
     </joint>
     <xacro:include filename="$(find xarm_description)/urdf/xarm_device_macro.xacro"/>
-    <xacro:xarm_device robot_type="lite" dof="6"
+    <xacro:xarm_device robot_type="${'lite' if robot == 'lite6' else 'xarm'}" dof="6"
       attach_to="platform_link" create_attach_link="false"
       attach_xyz="${' '.join(map(str, arm['xyz']))}"
@@ -54,23 +67,34 @@
       ros2_control_params="${'$(find amiga_arm_description)/config/sim_controllers.yaml' if gripper else ''}"
       robot_ip="${robot_ip}"/>
-    <!-- Gripper Lite: xarm's links and joints, but not its add_gripper. That one makes finger 2
-         follow finger 1 through a Gazebo Classic style plugin that does not load in gz sim, so
-         here gz_ros2_control mimics finger_joint2 (its URDF <mimic>) instead. -->
+    <!-- Gripper, not through xarm's add_gripper: that one makes the fingers follow each other
+         through a Gazebo Classic style plugin that does not load in gz sim, and its position
+         control did not move the fingers reliably. Here both fingers are effort controlled, so
+         each squeezes with the commanded force, capped by its joint effort limit. They close
+         independently: gz_ros2_control's mimic did not follow an effort controlled finger, and a
+         velocity controlled one squeezed only as hard as the leaves resisted its speed.
+         lite6: xarm's Gripper Lite links (5 N). xarm6: the xArm Gripper as parallel jaws (30 N). -->
     <xacro:if value="${gripper}">
       <xacro:include filename="$(find xarm_description)/urdf/common/common.link.xacro"/>
-      <xacro:include filename="$(find xarm_description)/urdf/gripper/uflite_gripper.urdf.xacro"/>
-      <xacro:uflite_gripper_urdf attach_to="link_eef"/>
+      <xacro:if value="${robot == 'lite6'}">
+        <xacro:include filename="$(find xarm_description)/urdf/gripper/uflite_gripper.urdf.xacro"/>
+        <xacro:uflite_gripper_urdf attach_to="link_eef"/>
+      </xacro:if>
+      <xacro:if value="${robot == 'xarm6'}">
+        <xacro:include filename="$(find amiga_arm_description)/urdf/xarm_gripper_jaws.xacro"/>
+        <xacro:xarm_gripper_jaws attach_to="link_eef"/>
+      </xacro:if>
       <xacro:if value="${ros2_control_plugin == 'gz_ros2_control/GazeboSimSystem'}">
-        <ros2_control name="GripperLiteSystem" type="system">
+        <ros2_control name="GripperSystem" type="system">
           <hardware><plugin>${ros2_control_plugin}</plugin></hardware>
-          <joint name="finger_joint1">
-            <command_interface name="position"/>
-            <command_interface name="velocity"/>
-            <state_interface name="position"/>
-            <state_interface name="velocity"/>
-          </joint>
-          <joint name="finger_joint2">
-            <state_interface name="position"/>
-          </joint>
+          <!-- mimic="false": the gripper URDFs make finger_joint2 mimic finger_joint1 -->
+          <xacro:macro name="finger_joint" params="name">
+            <joint name="${name}" mimic="false">
+              <command_interface name="effort"/>
+              <state_interface name="position"/>
+              <state_interface name="velocity"/>
+            </joint>
+          </xacro:macro>
+          <xacro:finger_joint name="finger_joint1"/>
+          <xacro:finger_joint name="finger_joint2"/>
         </ros2_control>
       </xacro:if>
