Commit message: Draw the camera's mounting tube
A grey box under the front cross tube, running forward past the
camera; size and pose in arm_platform.yaml next to the camera pose.
Visual only, so it never touches Plants.

File: src/amiga_arm_description/urdf/oak_camera.xacro (robot description, xacro)
@@ -14,4 +14,16 @@
       cam_pos_x="${cam['xyz'][0]}" cam_pos_y="${cam['xyz'][1]}" cam_pos_z="${cam['xyz'][2]}"
       cam_roll="${cam['rpy'][0]}" cam_pitch="${cam['rpy'][1]}" cam_yaw="${cam['rpy'][2]}"/>
+    <!-- The camera's mounting tube, visual only: no collision, so it never touches Plants -->
+    <link name="oak_tube_link">
+      <visual>
+        <geometry><box size="${' '.join(map(str, cam['tube']['size']))}"/></geometry>
+        <material name="amiga_grey"/>
+      </visual>
+    </link>
+    <joint name="oak_tube_joint" type="fixed">
+      <parent link="${parent}"/>
+      <child link="oak_tube_link"/>
+      <origin xyz="${' '.join(map(str, cam['tube']['xyz']))}"/>
+    </joint>
     <xacro:if value="${gazebo}">
       <gazebo reference="oak_rgb_camera_frame">
